File: con.sch (KiCad schematic (older format))
At the start: 3 parts, among them P501 USB_OTG, X501 CON_SWD, X502 SUB-D9

Commit message: set subd9 pin 3 to gnd, correct solder mask margin
Connections:
- net GND: now also X502.3
- no-connect marks 10 -> 9
Changed lines of the file:
@@
 NoConn ~ 5700 3450
 NoConn ~ 7700 2700
-NoConn ~ 7700 2900
 NoConn ~ 7700 3000
 NoConn ~ 7700 3100
@@
 	3900 2900 4000 2900
 NoConn ~ 4000 3200
+$Comp
+L GND #PWR?
+U 1 1 56F8617B
+P 7700 2900
+F 0 "#PWR?" H 7700 2650 50  0001 C CNN
+F 1 "GND" H 7700 2750 50  0000 C CNN
+F 2 "" H 7700 2900 50  0000 C CNN
+F 3 "" H 7700 2900 50  0000 C CNN
+	1    7700 2900
+	0    1    1    0
+$EndComp
 $EndSCHEMATC
