File: CAN.sch (KiCad schematic (older format))
At the start: 6 parts, among them U401 TJA1051/3

Commit message: remove unneeded parts
Parts:
- removed C401: 10uF, Capacitors_SMD:C_0805, symbol C_Small
Changed lines of the file:
@@
-$EndComp
-$Comp
-L C_Small C401
-U 1 1 56F5A553
-P 5400 4650
-F 0 "C401" H 5410 4720 50  0000 L CNN
-F 1 "10uF" H 5410 4570 50  0000 L CNN
-F 2 "Capacitors_SMD:C_0805" H 5400 4650 50  0001 C CNN
-F 3 "" H 5400 4650 50  0000 C CNN
-	1    5400 4650
-	1    0    0    -1
-$EndComp
-$Comp
-L GND #PWR022
-U 1 1 56F5A5CA
-P 5400 4750
-F 0 "#PWR022" H 5400 4500 50  0001 C CNN
-F 1 "GND" H 5400 4600 50  0000 C CNN
-F 2 "" H 5400 4750 50  0000 C CNN
-F 3 "" H 5400 4750 50  0000 C CNN
-	1    5400 4750
-	1    0    0    -1
 $EndComp
 $Comp
@@
 	1    0    0    -1
 $EndComp
-$Comp
-L +5V #PWR026
-U 1 1 56F5A9CA
-P 5400 4550
-F 0 "#PWR026" H 5400 4400 50  0001 C CNN
-F 1 "+5V" H 5400 4690 50  0000 C CNN
-F 2 "" H 5400 4550 50  0000 C CNN
-F 3 "" H 5400 4550 50  0000 C CNN
-	1    5400 4550
-	1    0    0    -1
-$EndComp

Commit message: add testpoints, reset line cap
Parts:
- R402: footprint Resistors_SMD:R_0603 -> Resistors_SMD:R_0805
Changed lines of the file:
@@
 CAN_L
 $Comp
-L GND #PWR021
+L GND #PWR024
 U 1 1 56F59A07
 P 5200 4000
-F 0 "#PWR021" H 5200 3750 50  0001 C CNN
+F 0 "#PWR024" H 5200 3750 50  0001 C CNN
 F 1 "GND" H 5200 3850 50  0000 C CNN
 F 2 "" H 5200 4000 50  0000 C CNN
@@
 $EndComp
 $Comp
-L GND #PWR023
+L GND #PWR025
 U 1 1 56F5A5EA
 P 5700 4750
-F 0 "#PWR023" H 5700 4500 50  0001 C CNN
+F 0 "#PWR025" H 5700 4500 50  0001 C CNN
 F 1 "GND" H 5700 4600 50  0000 C CNN
 F 2 "" H 5700 4750 50  0000 C CNN
@@
 $EndComp
 $Comp
-L GND #PWR024
+L GND #PWR026
 U 1 1 56F5A60A
 P 6000 4750
-F 0 "#PWR024" H 6000 4500 50  0001 C CNN
+F 0 "#PWR026" H 6000 4500 50  0001 C CNN
 F 1 "GND" H 6000 4600 50  0000 C CNN
 F 2 "" H 6000 4750 50  0000 C CNN
@@
 $EndComp
 $Comp
-L +3V3 #PWR025
+L +3V3 #PWR027
 U 1 1 56F5A80B
 P 6000 4550
-F 0 "#PWR025" H 6000 4400 50  0001 C CNN
+F 0 "#PWR027" H 6000 4400 50  0001 C CNN
 F 1 "+3V3" H 6000 4690 50  0000 C CNN
 F 2 "" H 6000 4550 50  0000 C CNN
@@
 $EndComp
 $Comp
-L +5V #PWR027
+L +5V #PWR028
 U 1 1 56F5A9E6
 P 5700 4550
-F 0 "#PWR027" H 5700 4400 50  0001 C CNN
+F 0 "#PWR028" H 5700 4400 50  0001 C CNN
 F 1 "+5V" H 5700 4690 50  0000 C CNN
 F 2 "" H 5700 4550 50  0000 C CNN
@@
 $EndComp
 $Comp
-L +3V3 #PWR028
+L +3V3 #PWR029
 U 1 1 56F5AB59
 P 5200 3700
-F 0 "#PWR028" H 5200 3550 50  0001 C CNN
+F 0 "#PWR029" H 5200 3550 50  0001 C CNN
 F 1 "+3V3" H 5200 3840 50  0000 C CNN
 F 2 "" H 5200 3700 50  0000 C CNN
@@
 $EndComp
 $Comp
-L +5V #PWR029
+L +5V #PWR030
 U 1 1 56F5AB75
 P 5200 3500
-F 0 "#PWR029" H 5200 3350 50  0001 C CNN
+F 0 "#PWR030" H 5200 3350 50  0001 C CNN
 F 1 "+5V" H 5200 3640 50  0000 C CNN
 F 2 "" H 5200 3500 50  0000 C CNN
@@
 Connection ~ 4550 3300
 $Comp
-L +3V3 #PWR030
+L +3V3 #PWR031
 U 1 1 56F69C59
 P 4550 2950
-F 0 "#PWR030" H 4550 2800 50  0001 C CNN
+F 0 "#PWR031" H 4550 2800 50  0001 C CNN
 F 1 "+3V3" H 4550 3090 50  0000 C CNN
 F 2 "" H 4550 2950 50  0000 C CNN
@@
 F 0 "R402" V 6730 3150 50  0000 C CNN
 F 1 "dnp" V 6650 3150 50  0000 C CNN
-F 2 "Resistors_SMD:R_0603" V 6580 3150 50  0001 C CNN
+F 2 "Resistors_SMD:R_0805" V 6580 3150 50  0001 C CNN
 F 3 "" H 6650 3150 50  0000 C CNN
 	1    6650 3150
