File: candleLight.sch (KiCad schematic (older format))
At the start: 0 parts

Commit message: add fiducials
Parts:
- added FID101, FID102, FID?: Dummy_FIDUCIAL_Passermarke_Type1_RevE_Date16Nov20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, Fiducials:Fiducial_1mm_Dia_2.54mm_Outer_CopperTop, symbol Dummy_FIDUCIAL_Passermarke_Type1_RevE_Date16Nov2011
Changed lines of the file:
@@
 LIBS:micro-usb-ab
 LIBS:con_swd
+LIBS:SymbolsSimilarEN60617+oldDIN617-RevE8
 LIBS:candleLight-cache
 EELAYER 25 0
@@
 Wire Wire Line
 	4150 5500 4700 5500
+$Comp
+L Dummy_FIDUCIAL_Passermarke_Type1_RevE_Date16Nov2011 FID101
+U 1 1 56FC5CD2
+P 9900 950
+F 0 "FID101" H 9900 1100 50  0000 C CNN
+F 1 "Dummy_FIDUCIAL_Passermarke_Type1_RevE_Date16Nov2011" H 9900 800 50  0000 C CNN
+F 2 "Fiducials:Fiducial_1mm_Dia_2.54mm_Outer_CopperTop" H 9900 950 50  0001 C CNN
+F 3 "" H 9900 950 50  0000 C CNN
+	1    9900 950
+	1    0    0    -1
+$EndComp
+$Comp
+L Dummy_FIDUCIAL_Passermarke_Type1_RevE_Date16Nov2011 FID102
+U 1 1 56FC5DC9
+P 9900 1350
+F 0 "FID102" H 9900 1500 50  0000 C CNN
+F 1 "Dummy_FIDUCIAL_Passermarke_Type1_RevE_Date16Nov2011" H 9900 1200 50  0000 C CNN
+F 2 "Fiducials:Fiducial_1mm_Dia_2.54mm_Outer_CopperTop" H 9900 1350 50  0001 C CNN
+F 3 "" H 9900 1350 50  0000 C CNN
+	1    9900 1350
+	1    0    0    -1
+$EndComp
+$Comp
+L Dummy_FIDUCIAL_Passermarke_Type1_RevE_Date16Nov2011 FID?
+U 1 1 56FC6D4E
+P 9900 1750
+F 0 "FID?" H 9900 1900 50  0000 C CNN
+F 1 "Dummy_FIDUCIAL_Passermarke_Type1_RevE_Date16Nov2011" H 9900 1600 50  0000 C CNN
+F 2 "Fiducials:Fiducial_1mm_Dia_2.54mm_Outer_CopperTop" H 9900 1750 50  0001 C CNN
+F 3 "" H 9900 1750 50  0000 C CNN
+	1    9900 1750
+	1    0    0    -1
+$EndComp
 $EndSCHEMATC

Commit message: add testpoints, reset line cap
Parts:
- gave numbers to parts that had none: 1
Changed lines of the file:
@@
 $EndComp
 $Comp
-L Dummy_FIDUCIAL_Passermarke_Type1_RevE_Date16Nov2011 FID?
+L Dummy_FIDUCIAL_Passermarke_Type1_RevE_Date16Nov2011 FID103
 U 1 1 56FC6D4E
 P 9900 1750
-F 0 "FID?" H 9900 1900 50  0000 C CNN
+F 0 "FID103" H 9900 1900 50  0000 C CNN
 F 1 "Dummy_FIDUCIAL_Passermarke_Type1_RevE_Date16Nov2011" H 9900 1600 50  0000 C CNN
 F 2 "Fiducials:Fiducial_1mm_Dia_2.54mm_Outer_CopperTop" H 9900 1750 50  0001 C CNN
