File: candleLight.kicad_pcb (KiCad board)
At the start: 2 copper layers, 37.7 x 20 mm, 44 parts, among them P501 USB_OTG, U201 STM32F072C8Tx, U301 MCP1754ST-3302E/MB, U401 TJA1051/3, X501 CON_SWD, X502 SUB-D9, Y201 8MHz

Commit message: optimize
Routing:
- net /MCU/CAN_RX: track 16.0 -> 15.5 mm
Other:
- board text added: "B"
- board text added: "T"
Changed lines of the file:
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@@
     (area 41.324999 74.924999 79.175001 95.075001)
     (thickness 1.6)
-    (drawings 22)
-    (tracks 467)
+    (drawings 23)
+    (tracks 466)
     (zones 0)
     (modules 44)
@@
   )
   (setup
-    (last_trace_width 0.15)
+    (last_trace_width 0.25)
     (user_trace_width 0.15)
     (trace_clearance 0.15)
@@
     (tags "Mesurement Point Round SMD Pad 1.5mm")
     (attr virtual)
-    (fp_text reference SCL (at -2.25 0.25) (layer B.SilkS)
+    (fp_text reference SCL (at -0.55 -1.55) (layer B.SilkS)
       (effects (font (size 1 1) (thickness 0.25)) (justify mirror))
     )
@@
     (tags "Mesurement Point Round SMD Pad 1.5mm")
     (attr virtual)
-    (fp_text reference SDA (at 2.3 0.2) (layer B.SilkS)
+    (fp_text reference SDA (at 0.7 -1.55) (layer B.SilkS)
       (effects (font (size 1 1) (thickness 0.25)) (justify mirror))
     )
@@
       (net 17 /CAN/CAN_L))
   )
+  (gr_text T (at 71.7 85.5 90) (layer F.SilkS)
+    (effects (font (size 1 1) (thickness 0.25)))
+  )
+  (gr_text B (at 57.6 92.9 90) (layer F.SilkS)
+    (effects (font (size 1 1) (thickness 0.25)))
+  )
   (dimension 19.95 (width 0.25) (layer Dwgs.User)
     (gr_text "19,950 mm" (at 37.65 84.975 270) (layer Dwgs.User)
@@
     (effects (font (size 1 1) (thickness 0.25)) (justify mirror))
   )
-  (gr_text CAN_H (at 71.2 86.7) (layer B.SilkS)
+  (gr_text CAN_H (at 71.2 86.5) (layer B.SilkS)
     (effects (font (size 1 1) (thickness 0.25)) (justify mirror))
   )
-  (gr_text +5V (at 48.45 75.95) (layer B.SilkS)
+  (gr_text +5V (at 48.6 76.1) (layer B.SilkS)
     (effects (font (size 1 1) (thickness 0.25)) (justify mirror))
   )
-  (gr_text GND (at 44.25 75.95) (layer B.SilkS)
+  (gr_text GND (at 44.25 76.1) (layer B.SilkS)
     (effects (font (size 1 1) (thickness 0.25)) (justify mirror))
   )
   (gr_line (start 41.4 75) (end 41.4 81.1) (layer Edge.Cuts) (width 0.15))
   (gr_line (start 79.1 75) (end 79.1 95) (layer Edge.Cuts) (width 0.15))
-  (gr_circle (center 61.3 88.8) (end 61.4 88.9) (layer F.SilkS) (width 0.2))
   (gr_line (start 47 81.9) (end 47 88.1) (angle 90) (layer Edge.Cuts) (width 0.15))
   (gr_line (start 41.4 81.1) (end 46.2 81.1) (angle 90) (layer Edge.Cuts) (width 0.15))
@@
   (segment (start 68.049999 85.100001) (end 68.5 84.65) (width 0.25) (layer F.Cu) (net 3))
   (segment (start 64.175 86) (end 64.15 86) (width 0.25) (layer F.Cu) (net 3))
+  (segment (start 57.45 83.8) (end 56.075001 83.8) (width 0.25) (layer F.Cu) (net 4))
+  (segment (start 60.703184 87.053184) (end 57.45 83.8) (width 0.25) (layer F.Cu) (net 4))
+  (segment (start 60.703184 87.84906) (end 60.703184 87.053184) (width 0.25) (layer F.Cu) (net 4))
+  (segment (start 61.15 89.05) (end 61.15 88.295876) (width 0.25) (layer F.Cu) (net 4))
+  (segment (start 61.15 88.295876) (end 60.703184 87.84906) (width 0.25) (layer F.Cu) (net 4))
   (segment (start 57.6 93.85) (end 57.6 92.963182) (width 0.25) (layer F.Cu) (net 4))
   (segment (start 57.6 92.963182) (end 57.824148 92.739034) (width 0.25) (layer F.Cu) (net 4))
@@
   (segment (start 58.525001 92.520001) (end 58.525001 92.3) (width 0.25) (layer F.Cu) (net 4))
   (segment (start 58.525001 92.3) (end 59.35 92.3) (width 0.25) (layer F.Cu) (net 4))
-  (segment (start 60.703184 87.053184) (end 57.45 83.8) (width 0.25) (layer F.Cu) (net 4))
-  (segment (start 60.703184 88.01691) (end 60.703184 87.053184) (width 0.25) (layer F.Cu) (net 4))
-  (segment (start 61.15 89.05) (end 61.15 88.463726) (width 0.25) (layer F.Cu) (net 4))
-  (segment (start 61.15 88.463726) (end 60.703184 88.01691) (width 0.25) (layer F.Cu) (net 4))
-  (segment (start 57.45 83.8) (end 56.075001 83.8) (width 0.25) (layer F.Cu) (net 4))
   (segment (start 56.075001 85.924999) (end 56.075001 83.8) (width 0.25) (layer F.Cu) (net 4))
   (segment (start 56.075001 83.8) (end 56.075001 81.875001) (width 0.25) (layer F.Cu) (net 4))
@@
   (segment (start 71.65 77.4) (end 69.00052 77.4) (width 0.25) (layer F.Cu) (net 4))
   (segment (start 69.00052 77.4) (end 68.90166 77.49886) (width 0.25) (layer F.Cu) (net 4))
-  (segment (start 48.3 82.5) (end 48.3 78.65) (width 0.25) (layer B.Cu) (net 5))
+  (segment (start 48.3 82.5) (end 48.3 78.65) (width 0.4) (layer B.Cu) (net 5))
   (segment (start 48.3 78.65) (end 48.15 78.5) (width 0.25) (layer B.Cu) (net 5))
-  (segment (start 47.875 83.7) (end 47.875 82.925) (width 0.25) (layer F.Cu) (net 5))
-  (segment (start 47.875 82.925) (end 48.3 82.5) (width 0.25) (layer F.Cu) (net 5))
+  (segment (start 47.875 83.7) (end 47.875 82.925) (width 0.4) (layer F.Cu) (net 5))
+  (segment (start 47.875 82.925) (end 48.3 82.5) (width 0.4) (layer F.Cu) (net 5))
   (via (at 48.3 82.5) (size 0.6) (drill 0.4) (layers F.Cu B.Cu) (net 5))
   (segment (start 70.45 88.447119) (end 66.767265 92.129854) (width 0.25) (layer B.Cu) (net 5))
@@
   (segment (start 65.1 92.435) (end 62.985 92.435) (width 0.25) (layer F.Cu) (net 5))
   (segment (start 62.985 92.435) (end 62.85 92.3) (width 0.25) (layer F.Cu) (net 5))
-  (segment (start 72.8 81.05) (end 71.65 81.05) (width 0.25) (layer F.Cu) (net 5))
-  (segment (start 72.8 76.05) (end 72.8 81.05) (width 0.25) (layer B.Cu) (net 5))
+  (segment (start 72.8 81.05) (end 71.65 81.05) (width 0.4) (layer F.Cu) (net 5))
+  (segment (start 72.8 76.05) (end 72.8 81.05) (width 0.4) (layer B.Cu) (net 5))
   (via (at 72.8 81.05) (size 0.6) (drill 0.4) (layers F.Cu B.Cu) (net 5))
   (segment (start 72.75 76) (end 72.8 76.05) (width 0.25) (layer B.Cu) (net 5))
-  (segment (start 69.5 76) (end 72.75 76) (width 0.25) (layer B.Cu) (net 5))
-  (segment (start 48.52868 76) (end 69.5 76) (width 0.25) (layer B.Cu) (net 5))
-  (segment (start 48.15 78.5) (end 48.15 76.37868) (width 0.25) (layer B.Cu) (net 5))
-  (segment (start 48.15 76.37868) (end 48.52868 76) (width 0.25) (layer B.Cu) (net 5))
+  (segment (start 69.5 76) (end 72.75 76) (width 0.4) (layer B.Cu) (net 5))
+  (segment (start 48.52868 76) (end 69.5 76) (width 0.4) (layer B.Cu) (net 5))
+  (segment (start 48.15 78.5) (end 48.15 76.37868) (width 0.4) (layer B.Cu) (net 5))
+  (segment (start 48.15 76.37868) (end 48.52868 76) (width 0.4) (layer B.Cu) (net 5))
   (segment (start 48 78.65) (end 48.15 78.5) (width 0.25) (layer B.Cu) (net 5))
   (segment (start 60.35 77.0007) (end 61.8493 77.0007) (width 0.25) (layer F.Cu) (net 6))
@@
   (segment (start 49.590713 94.028699) (end 46.863699 94.028699) (width 0.25) (layer F.Cu) (net 26))
   (segment (start 46.863699 94.028699) (end 46.47 93.635) (width 0.25) (layer F.Cu) (net 26))
-  (segment (start 63.529087 87.329087) (end 59.291251 87.329087) (width 0.25) (layer B.Cu) (net 27))
-  (segment (start 66.7 90.5) (end 63.529087 87.329087) (width 0.25) (layer B.Cu) (net 27))
-  (segment (start 59.291251 87.329087) (end 58.991252 87.629086) (width 0.25) (layer B.Cu) (net 27))
-  (segment (start 58.6 88.020338) (end 58.691253 87.929085) (width 0.25) (layer F.Cu) (net 27))
-  (segment (start 58.6 89.55) (end 58.6 88.020338) (width 0.25) (layer F.Cu) (net 27))
-  (via (at 58.991252 87.629086) (size 0.6) (drill 0.4) (layers F.Cu B.Cu) (net 27))
-  (segment (start 58.691253 87.929085) (end 58.991252 87.629086) (width 0.25) (layer F.Cu) (net 27))
+  (segment (start 58.6 88.351134) (end 58.461607 88.212741) (width 0.25) (layer F.Cu) (net 27))
+  (segment (start 58.6 89.55) (end 58.6 88.351134) (width 0.25) (layer F.Cu) (net 27))
+  (segment (start 58.461607 88.385871) (end 58.461607 88.212741) (width 0.25) (layer B.Cu) (net 27))
+  (segment (start 60.575736 90.5) (end 58.461607 88.385871) (width 0.25) (layer B.Cu) (net 27))
+  (segment (start 61 90.5) (end 60.575736 90.5) (width 0.25) (layer B.Cu) (net 27))
+  (via (at 58.461607 88.212741) (size 0.6) (drill 0.4) (layers F.Cu B.Cu) (net 27))
+  (segment (start 66.7 90.5) (end 61 90.5) (width 0.25) (layer F.Cu) (net 27))
+  (via (at 61 90.5) (size 0.6) (drill 0.4) (layers F.Cu B.Cu) (net 27))
   (segment (start 66.125 93.705) (end 65.1 93.705) (width 0.25) (layer F.Cu) (net 27))
   (segment (start 67.081733 90.881733) (end 67.081733 92.748267) (width 0.25) (layer F.Cu) (net 27))
   (segment (start 66.7 90.5) (end 67.081733 90.881733) (width 0.25) (layer F.Cu) (net 27))
   (segment (start 67.081733 92.748267) (end 66.125 93.705) (width 0.25) (layer F.Cu) (net 27))
-  (via (at 66.7 90.5) (size 0.6) (drill 0.4) (layers F.Cu B.Cu) (net 27))
-  (segment (start 59.959265 88.222267) (end 59.535001 88.222267) (width 0.25) (layer B.Cu) (net 28))
-  (segment (start 59.972267 88.222267) (end 59.959265 88.222267) (width 0.25) (layer B.Cu) (net 28))
-  (segment (start 61.65 89.9) (end 59.972267 88.222267) (width 0.25) (layer B.Cu) (net 28))
-  (segment (start 59.1 88.65) (end 59.527733 88.222267) (width 0.25) (layer F.Cu) (net 28))
-  (segment (start 59.527733 88.222267) (end 59.535001 88.222267) (width 0.25) (layer F.Cu) (net 28))
-  (segment (start 59.1 89.55) (end 59.1 88.65) (width 0.25) (layer F.Cu) (net 28))
-  (via (at 59.535001 88.222267) (size 0.6) (drill 0.4) (layers F.Cu B.Cu) (net 28))
+  (segment (start 59.1 89.55) (end 59.1 88.351022) (width 0.25) (layer F.Cu) (net 28))
+  (segment (start 60.925984 89.9) (end 59.538502 88.512518) (width 0.25) (layer B.Cu) (net 28))
+  (segment (start 59.1 88.351022) (end 59.238503 88.212519) (width 0.25) (layer F.Cu) (net 28))
+  (segment (start 59.538502 88.512518) (end 59.238503 88.212519) (width 0.25) (layer B.Cu) (net 28))
+  (via (at 59.238503 88.212519) (size 0.6) (drill 0.4) (layers F.Cu B.Cu) (net 28))
+  (segment (start 61.65 89.9) (end 60.925984 89.9) (width 0.25) (layer B.Cu) (net 28))
   (segment (start 61.65 89.9) (end 65.095 89.9) (width 0.25) (layer F.Cu) (net 28))
   (segment (start 65.095 89.9) (end 65.1 89.895) (width 0.25) (layer F.Cu) (net 28))

Commit message: fine tuning
Parts:
- moved Y201 0.25 mm to (68.5, 85.2)
Routing:
- net GND: track 154.8 -> 147.5 mm, vias 22 -> 24
- net /LEDs/LED2: track 8.34 -> 9.60 mm
- net Net-(C201-Pad2): track 9.38 -> 8.17 mm
- net Net-(U201-Pad25): track 5.14 -> 6.27 mm
- net +3V3: track 115.2 -> 116.2 mm
- net /Connectors/SWCLK: track 10.1 -> 11.0 mm

Commit message: v1.1
Parts:
- X502: footprint Connect:DB9M_CI -> subd9:DB9M_CI
Routing:
- net GND: track 147.5 -> 148.8 mm
- net +3V3: track 116.2 -> 117.3 mm
