File: power.sch (KiCad schematic (older format))
At the start: 3 parts, among them U301 MCP1754ST-3302E/MB

Commit message: add testpoints, reset line cap
Parts:
- added W301, W302, W303: TEST_1P, Measurement_Points:Measurement_Point_Round-SMD-Pad_Big, symbol TEST_1P
Connections:
- net +3V3: now also W303.1
- net +5V: now also W301.1
- net GND: now also W302.1
Other:
- moved on the sheet: C301
Changed lines of the file:
@@
 $EndComp
 $Comp
-L GND #PWR018
+L GND #PWR019
 U 1 1 56F60A54
 P 5650 4300
-F 0 "#PWR018" H 5650 4050 50  0001 C CNN
+F 0 "#PWR019" H 5650 4050 50  0001 C CNN
 F 1 "GND" H 5650 4150 50  0000 C CNN
 F 2 "" H 5650 4300 50  0000 C CNN
@@
 $EndComp
 $Comp
-L +5V #PWR019
+L +5V #PWR020
 U 1 1 56F60A70
-P 5000 3750
-F 0 "#PWR019" H 5000 3600 50  0001 C CNN
-F 1 "+5V" H 5000 3890 50  0000 C CNN
-F 2 "" H 5000 3750 50  0000 C CNN
-F 3 "" H 5000 3750 50  0000 C CNN
-	1    5000 3750
+P 4900 3750
+F 0 "#PWR020" H 4900 3600 50  0001 C CNN
+F 1 "+5V" H 4900 3890 50  0000 C CNN
+F 2 "" H 4900 3750 50  0000 C CNN
+F 3 "" H 4900 3750 50  0000 C CNN
+	1    4900 3750
 	0    -1   -1   0
 $EndComp
 $Comp
-L +3V3 #PWR020
+L +3V3 #PWR021
 U 1 1 56F60A9D
 P 6400 3750
-F 0 "#PWR020" H 6400 3600 50  0001 C CNN
+F 0 "#PWR021" H 6400 3600 50  0001 C CNN
 F 1 "+3V3" H 6400 3890 50  0000 C CNN
 F 2 "" H 6400 3750 50  0000 C CNN
@@
 L C_Small C301
 U 1 1 56F60BBB
-P 5200 3950
-F 0 "C301" H 5210 4020 50  0000 L CNN
-F 1 "10uF" H 5210 3870 50  0000 L CNN
-F 2 "Capacitors_SMD:C_0805" H 5200 3950 50  0001 C CNN
-F 3 "" H 5200 3950 50  0000 C CNN
-	1    5200 3950
+P 5100 3950
+F 0 "C301" H 5110 4020 50  0000 L CNN
+F 1 "10uF" H 5110 3870 50  0000 L CNN
+F 2 "Capacitors_SMD:C_0805" H 5100 3950 50  0001 C CNN
+F 3 "" H 5100 3950 50  0000 C CNN
+	1    5100 3950
 	1    0    0    -1
 $EndComp
@@
 Wire Wire Line
 	6150 3850 6150 3750
-Wire Wire Line
-	5650 3950 5650 4300
 Connection ~ 5650 4150
 Wire Wire Line
@@
 Connection ~ 6150 4150
 Wire Wire Line
-	5000 3750 5350 3750
+	4900 3750 5350 3750
 Wire Wire Line
-	5200 3850 5200 3750
-Connection ~ 5200 3750
+	5100 3850 5100 3750
+Connection ~ 5100 3750
 Wire Wire Line
-	5200 4050 5200 4150
+	5100 4050 5100 4150
 Wire Wire Line
-	5200 4150 6150 4150
+	5100 4150 6150 4150
 Wire Wire Line
 	5950 3750 6400 3750
 Connection ~ 6150 3750
+$Comp
+L TEST_1P W301
+U 1 1 57223B24
+P 5100 3750
+F 0 "W301" H 5100 4020 50  0000 C CNN
+F 1 "TEST_1P" H 5100 3950 50  0000 C CNN
+F 2 "Measurement_Points:Measurement_Point_Round-SMD-Pad_Big" H 5300 3750 50  0001 C CNN
+F 3 "" H 5300 3750 50  0000 C CNN
+	1    5100 3750
+	1    0    0    -1
+$EndComp
+$Comp
+L TEST_1P W302
+U 1 1 57223B69
+P 5100 4150
+F 0 "W302" H 5100 4420 50  0000 C CNN
+F 1 "TEST_1P" H 5100 4350 50  0000 C CNN
+F 2 "Measurement_Points:Measurement_Point_Round-SMD-Pad_Big" H 5300 4150 50  0001 C CNN
+F 3 "" H 5300 4150 50  0000 C CNN
+	1    5100 4150
+	-1   0    0    1
+$EndComp
+$Comp
+L TEST_1P W303
+U 1 1 572267AA
+P 6150 3750
+F 0 "W303" H 6150 4020 50  0000 C CNN
+F 1 "TEST_1P" H 6150 3950 50  0000 C CNN
+F 2 "Measurement_Points:Measurement_Point_Round-SMD-Pad_Big" H 6350 3750 50  0001 C CNN
+F 3 "" H 6350 3750 50  0000 C CNN
+	1    6150 3750
+	1    0    0    -1
+$EndComp
+Wire Wire Line
+	5650 3950 5650 4300
+Connection ~ 5100 4150
+$Comp
+L GND #PWR022
+U 1 1 57229925
+P 3150 4050
+F 0 "#PWR022" H 3150 3800 50  0001 C CNN
+F 1 "GND" H 3150 3900 50  0000 C CNN
+F 2 "" H 3150 4050 50  0000 C CNN
+F 3 "" H 3150 4050 50  0000 C CNN
+	1    3150 4050
+	1    0    0    -1
+$EndComp
+$Comp
+L PWR_FLAG #FLG023
+U 1 1 57229968
+P 3150 4050
+F 0 "#FLG023" H 3150 4145 50  0001 C CNN
+F 1 "PWR_FLAG" H 3150 4230 50  0000 C CNN
+F 2 "" H 3150 4050 50  0000 C CNN
+F 3 "" H 3150 4050 50  0000 C CNN
+	1    3150 4050
+	1    0    0    -1
+$EndComp
 $EndSCHEMATC

Commit message: candleLight v1.2
Parts:
- removed W303: TEST_1P, Measurement_Points:Measurement_Point_Round-SMD-Pad_Big, symbol TEST_1P
Changed lines of the file:
@@
 	-1   0    0    1
-$EndComp
-$Comp
-L TEST_1P W303
-U 1 1 572267AA
-P 6150 3750
-F 0 "W303" H 6150 4020 50  0000 C CNN
-F 1 "TEST_1P" H 6150 3950 50  0000 C CNN
-F 2 "Measurement_Points:Measurement_Point_Round-SMD-Pad_Big" H 6350 3750 50  0001 C CNN
-F 3 "" H 6350 3750 50  0000 C CNN
-	1    6150 3750
-	1    0    0    -1
 $EndComp
 Wire Wire Line
